File: GoPack v2.0 - Pi 3 Simulink r2017b/GoPack Board Rev A/Pi MCU shield 2.sch (EAGLE design)
At the start: 60 parts, among them U1 DSPIC33FJ64MC204TQFP, U2 LMH6644MT, U3 LMH6644MT, U4 MC3846D, U5 UA9637AC, U6 LM25011, U7 5V Reg, U8 3V3 Reg, U9 LMH6644MT, X1 Supply, X2 Pwr Switch, X3 Motor Kill, X4 Motor Supply

Commit message: Adding Board Files
Parts:
- removed X3: Motor Kill, con-wago-500:W237-102
- removed X4: Motor Supply, con-wago-500:W237-102
- added C18, C36, C38: 100pF, SparkFun-Capacitors:CAP0603-CAP
- added C19, C37, C39: 47pF, SparkFun-Capacitors:CAP0603-CAP
- added CR1: SMBJ54A-E3/52, vishaydiode:SMBJ54A-E3/52
- added F1: 0157004.DR, lilfuse:0157004.DR
- added L2, L3, L4: DR127-220-R, wurth:DR127-220-R
- added R17, R18, R19: 1k, resistor:R-US_R0603
- added R20, R47, R48: 1200, resistor:R-US_R0603
- added R21, R22, R23, R24, R25, R26: 33k, resistor:R-US_R0603
- added U$1: MM438725438725, Misc:MM438725438725
- added X5: (no value), con-wago-508:W237-06P
- added X6: (no value), con-wago-508:W237-11P
- R14, R15, R16: value 50k -> 10k
- R2, R8: value 1k -> 150
- R3, R4: value 470 -> 82
Connections:
- removed net N$3: C8.1, C9.2, R12.2, U6.VIN, X2-2.KL, X3-1.KL
- removed net N$7: X3-2.KL, X4-1.KL
- new net N$11: C18.1, R20.2
- new net N$12: U$1.HALL_SENSOR_2, X6-6.KL
- new net N$13: U$1.HALL_SENSOR_3, X6-7.KL
- new net N$14: U$1.DIGIN1, X6-8.KL
- new net N$15: U$1.DIGIN2, X6-9.KL
- new net N$17: U$1.DIGIN/DIGOUT3, X6-10.KL
- new net N$19: U$1.DIGIN/DIGOUT4, X6-11.KL
- new net N$20: U$1.ANIN1+, X5-1.KL
- new net N$21: U$1.ANIN1-, X5-2.KL
- new net N$22: U$1.ANIN2+, X5-3.KL
- new net N$24: C36.2, C37.2, L2.1, X6-2.KL
- new net N$26: U$1.ANIN2-, X5-4.KL
- new net N$27: U$1.ANOUT1, X5-5.KL
- new net N$34: U$1.ANOUT2, X5-6.KL
- new net N$41: C36.1, R47.2
- new net N$6: C18.2, C19.2, L4.1, X6-1.KL
- new net N$62: C38.2, C39.2, L3.1, X6-3.KL
- new net N$64: C38.1, R48.2
- new net N$65: L2.2, U$1.MOTOR(-M)/MOTOR_WINDING2@3, U$1.MOTOR(-M)/MOTOR_WINDING2@4
- new net N$66: L3.2, U$1.MOTOR_WINDING3@5, U$1.MOTOR_WINDING3@6
- new net N$8: L4.2, U$1.MOTOR(+M)/MOTOR_WINDING@1, U$1.MOTOR(+M)/MOTOR_WINDING@2
- new net N$9: U$1.HALL_SENSOR_1, X6-5.KL
- new net PWR: C8.1, C9.2, CR1.12, F1.2, R12.2, U$1.+VCC@7, U$1.+VCC@8, U6.VIN
- new net PWR-PREFUSE: F1.1, X2-2.KL
- net !A1: now also R24.2
- net !A2: now also R22.1
- net !B1: now also R21.1
- net !B2: now also R25.1
- net !I1: now also R23.2
- net !I2: now also R26.1
- net +5V: now also U$1.+5VDC
- net A1: now also R24.1
- net A2: now also R22.2
- net B1: now also R21.2
- net B2: now also R25.2
- net GND: now also C19.1, C37.1, C39.1, CR1.21, R17.1, R18.1, R19.1, R20.1, R47.1, R48.1, U$1.GND, U$1.POWER_GND/GND@10, U$1.POWER_GND/GND@9; no longer R14.A, R15.A, R16.A, X4-2.KL
- net I1: now also R23.1
- net I2: now also R26.2
- net N$1: now also R18.2
- net N$10: now also R17.2
- net N$31: now also R19.2
Other:
- moved on the sheet: C16, C17, X1-1, X1-2, X2-1, X2-2
